File: Kicad/hydration_tracker/hydration_tracker.kicad_sch (KiCad schematic)
At the start: 11 parts, among them M1 Stepper_Motor_bipolar, SW1 PTS636 SM50 SMTR LFS, U1 ESP32C3, U7 ESP32C3

Commit message: add label
Parts:
- M1: footprint (none) -> Connector_PinHeader_2.54mm:PinHeader_1x04_P2.54mm_Vertical_SMD_Pin1Left
- SW1: footprint SW_PTS636_SMT-G_5_CNK -> footprints_PTS636:SW_PTS636_SMT-G_5_CNK
Changed lines of the file:
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@@
+		)
+	)
+	(label "Display Device"
+		(at 187.96 35.56 0)
+		(effects
+			(font
+				(size 1.27 1.27)
+			)
+			(justify left bottom)
+		)
+	)
+	(label "Sensor device"
+		(at 64.77 36.83 0)
+		(effects
+			(font
+				(size 1.27 1.27)
+			)
+			(justify left bottom)
 		)
 	)
@@
 			)
 		)
-		(property "Footprint" ""
+		(property "Footprint" "Connector_PinHeader_2.54mm:PinHeader_1x04_P2.54mm_Vertical_SMD_Pin1Left"
 			(at 162.306 68.834 0)
 			(effects
@@
 			)
 		)
-		(property "Footprint" "SW_PTS636_SMT-G_5_CNK"
+		(property "Footprint" "footprints_PTS636:SW_PTS636_SMT-G_5_CNK"
 			(at 208.28 77.47 0)
 			(effects

Commit message: finish sensor pcb
Parts:
- removed BT2: Battery, Connector_JST:JST_PH_S2B-PH-K_1x02_P2.00mm_Horizontal, symbol Device:Battery
- removed D1: NeoPixel_THT, LED_THT:LED_D5.0mm, symbol LED:NeoPixel_THT
- removed M1: Stepper_Motor_bipolar, Connector_PinHeader_2.54mm:PinHeader_1x04_P2.54mm_Vertical_SMD_Pin1Left, symbol Motor:Stepper_Motor_bipolar
- removed SW1: PTS636 SM50 SMTR LFS, footprints_PTS636:SW_PTS636_SMT-G_5_CNK, symbol 2026-01-27_02-22-24:PTS636_SM50_SMTR_LFS
- removed U1, U7: ESP32C3, RF_Module:ESP32-C3-DevKitM-1, symbol ESP32C3:ESP32C3
- added C1: 0.1uF, Capacitor_SMD:C_0805_2012Metric_Pad1.18x1.45mm_HandSolder, symbol Device:C
- added C2: 1uF, Capacitor_SMD:C_0805_2012Metric_Pad1.18x1.45mm_HandSolder, symbol Device:C
- added J1: RFShield_OnePiece, TestPoint:TestPoint_Pad_D1.0mm, symbol Device:RFShield_OnePiece
- added R1, R2: 4.7K, Resistor_SMD:R_0805_2012Metric_Pad1.20x1.40mm_HandSolder, symbol Device:R
- added U1: ~, GIX_ESP32:XIAO_ESP32, symbol GIX_ESP32:XIAO_ESP32
- added U7: FDC1004DGSR, footprints_FDC1004:DGS0010A_M, symbol 2026-01-30_07-42-30:FDC1004DGSR
Connections:
- net GND1 is gone; now on net GND2: BT1.2 (-)
- net +3V3: now also C1.2, C2.1, R1.2, R2.1, U1.12 (3V3), U7.8 (VDD)
- net GND2: now also C1.1, C2.2, U1.13 (GND), U1.16 (-BATT), U7.7 (GND)
- net VDD1 renamed VDD
- net VDD: now also U1.15 (+BATT)
- new net: U3.1, U7.4 (CIN3)
- new net: J1.1 (Shield), U7.1 (SHLD1), U7.6 (SHLD2)
- new net: U5.1, U7.2 (CIN1)
- new net: R2.2, U1.5 (GPIO4_A3_D3_SDA), U7.10 (SDA)
- new net: R1.1, U1.6 (GPIO6_A5_D5_SCL), U7.9 (SCL)
- new net: U6.1, U7.3 (CIN2)
- new net: U4.1, U7.5 (CIN4)
- no-connect marks 0 -> 10
